Commit message: Camera added

File: viratbot_description/urdf/viratbot.gazebo.xacro (robot description, xacro)
@@ -1,3 +1,40 @@
 <?xml version="1.0" encoding="UTF-8"?>
 <robot name="viratbot">
+    <!-- Camera Plugin -->
+    <gazebo reference="camera">
+        <sensor type="camera" name="camera1">
+            <update_rate>30.0</update_rate>
+            <camera name="head">
+                <horizontal_fov>1.3962634</horizontal_fov>
+                <image>
+                    <width>800</width>
+                    <height>800</height>
+                    <format>R8G8B8</format>
+                </image>
+                <clip>
+                    <near>0.02</near>
+                    <far>300</far>
+                </clip>
+                <noise>
+                    <type>gaussian</type>
+                    <mean>0.0</mean>
+                    <stddev>0.007</stddev>
+                </noise>
+            </camera>
+            <plugin name="camera_controller" filename="libgazebo_ros_camera.so">
+                <alwaysOn>true</alwaysOn>
+                <updateRate>0.0</updateRate>
+                <cameraName>viratbot/camera1</cameraName>
+                <imageTopicName>image_raw</imageTopicName>
+                <cameraInfoTopicName>camera_info</cameraInfoTopicName>
+                <frameName>camera</frameName>
+                <hackBaseline>0.07</hackBaseline>
+                <distortionK1>0.0</distortionK1>
+                <distortionK2>0.0</distortionK2>
+                <distortionK3>0.0</distortionK3>
+                <distortionT1>0.0</distortionT1>
+                <distortionT2>0.0</distortionT2>
+            </plugin>
+        </sensor>
+    </gazebo>
 </robot>

File: viratbot_description/urdf/viratbot.urdf.xacro (robot description, xacro)
@@ -1,9 +1,11 @@
 <?xml version="1.0"?>
 <robot name="viratbot" xmlns:xacro="http://www.ros.org/wiki/xacro">
-    <link name="base_link">
+    <xacro:include filename="$(find viratbot_description)/urdf/viratbot.gazebo.xacro"/>
+    <link name="base_link"></link>
+    <link name="chassis">
         <inertial>
-            <mass value="3"/>
-            <inertia ixx="0.05" ixy="0" ixz="0" iyy="0.17" iyz="0" izz="0.2"/>
-            <origin xyz="0 0 0.2" rpy="0 0 0"/>
+            <mass value="3" />
+            <inertia ixx="0.05" ixy="0" ixz="0" iyy="0.17" iyz="0" izz="0.2" />
+            <origin xyz="0 0 0.2" rpy="0 0 0" />
         </inertial>
         <collision>
@@ -32,7 +34,7 @@
         </visual>
         <visual>
-            <origin xyz="0.3 0 0.5" rpy="0 0 0" />
+            <origin xyz="0.3 0 0.43" rpy="0 0 0" />
             <geometry>
-                <cylinder radius="0.03" length="0.6" />
+                <cylinder radius="0.03" length="0.5" />
             </geometry>
         </visual>
@@ -40,7 +42,7 @@
     <link name="right_wheel">
         <inertial>
-            <mass value="0.3"/>
-            <inertia ixx="0.0325" ixy="0" ixz="0" iyy="0.006" iyz="0" izz="0.0325"/>
-            <origin xyz="0 0 0" rpy="0 1.5707 1.5707"/>
+            <mass value="0.3" />
+            <inertia ixx="0.0325" ixy="0" ixz="0" iyy="0.006" iyz="0" izz="0.0325" />
+            <origin xyz="0 0 0" rpy="0 1.5707 1.5707" />
         </inertial>
         <collision>
@@ -59,7 +61,7 @@
     <link name="left_wheel">
         <inertial>
-            <mass value="0.3"/>
-            <inertia ixx="0.0325" ixy="0" ixz="0" iyy="0.006" iyz="0" izz="0.0325"/>
-            <origin xyz="0 0 0" rpy="0 1.5707 1.5707"/>
+            <mass value="0.3" />
+            <inertia ixx="0.0325" ixy="0" ixz="0" iyy="0.006" iyz="0" izz="0.0325" />
+            <origin xyz="0 0 0" rpy="0 1.5707 1.5707" />
         </inertial>
         <collision>
@@ -76,6 +78,10 @@
         </visual>
     </link>
+    <joint name="base_chassis_joint" type="fixed">
+        <parent link="base_link" />
+        <child link="chassis" />
+    </joint>
     <joint name="right_wheel_hinge" type="continuous">
-        <parent link="base_link" />
+        <parent link="chassis" />
         <child link="right_wheel" />
         <axis xyz="0 1 0" />
@@ -83,8 +89,32 @@
     </joint>
     <joint name="left_wheel_hinge" type="continuous">
-        <parent link="base_link" />
+        <parent link="chassis" />
         <child link="left_wheel" />
         <axis xyz="0 1 0" />
         <origin xyz="-0.2 -0.26 0.2" rpy="0 0 0" />
     </joint>
+    <link name="camera">
+        <inertial>
+            <mass value="0.05" />
+            <inertia ixx="0.0005" ixy="0" ixz="0" iyy="0.0005" iyz="0" izz="0.0005" />
+        </inertial>
+        <collision>
+            <origin xyz="0 0 0" rpy="0 0 0" />
+            <geometry>
+                <box size="0.05 0.05 0.05" />
+            </geometry>
+        </collision>
+        <visual>
+            <origin xyz="0 0 0" rpy="0 0 0" />
+            <geometry>
+                <box size="0.05 0.05 0.05" />
+            </geometry>
+        </visual>
+    </link>
+    <joint name="camera_joint" type="fixed">
+        <axis xyz="0 0 1" />
+        <origin xyz="0.35 0 0.6" rpy="0 0.5 0" />
+        <parent link="chassis"/>
+        <child link="camera" />
+    </joint>
 </robot>

Commit message: Added diff drive

File: viratbot_description/urdf/viratbot.gazebo.xacro (robot description, xacro)
@@ -38,3 +38,23 @@
         </sensor>
     </gazebo>
+    <gazebo>
+        <plugin name="differential_drive_controller" filename="libgazebo_ros_diff_drive.so">
+          <updateRate>20</updateRate>
+          <leftJoint>left_wheel_hinge</leftJoint>
+          <rightJoint>right_wheel_hinge</rightJoint>
+          <wheelSeparation>0.52</wheelSeparation>
+          <wheelDiameter>0.4</wheelDiameter>
+          <wheelAcceleration>1.0</wheelAcceleration>
+          <wheelTorque>20</wheelTorque>
+          <commandTopic>cmd_vel</commandTopic>
+          <odometryTopic>odom</odometryTopic>
+          <odometryFrame>odom</odometryFrame>
+          <robotBaseFrame>base_link</robotBaseFrame>
+          <odometrySource>1</odometrySource>
+          <publishWheelTF>true</publishWheelTF>
+          <publishOdom>true</publishOdom>
+          <publishWheelJointState>true</publishWheelJointState>
+          <legacyMode>false</legacyMode>
+        </plugin>
+      </gazebo>
 </robot>

File: viratbot_description/urdf/viratbot.urdf.xacro (robot description, xacro)
@@ -1,5 +1,5 @@
 <?xml version="1.0"?>
 <robot name="viratbot" xmlns:xacro="http://www.ros.org/wiki/xacro">
-    <xacro:include filename="$(find viratbot_description)/urdf/viratbot.gazebo.xacro"/>
+    <xacro:include filename="$(find viratbot_description)/urdf/viratbot.gazebo.xacro" />
     <link name="base_link"></link>
     <link name="chassis">
@@ -7,5 +7,5 @@
             <mass value="3" />
             <inertia ixx="0.05" ixy="0" ixz="0" iyy="0.17" iyz="0" izz="0.2" />
-            <origin xyz="0 0 0.2" rpy="0 0 0" />
+            <origin xyz="0 0 0" rpy="0 0 0" />
         </inertial>
         <collision>
@@ -16,5 +16,5 @@
         </collision>
         <visual>
-            <origin rpy=" 0 0 0" xyz="0 0 0.2" />
+            <origin rpy=" 0 0 0" xyz="0 0 0" />
             <geometry>
                 <box size="0.8 0.4 0.2" />
@@ -22,5 +22,5 @@
         </visual>
         <collision>
-            <origin xyz="0.3 0 0.1" rpy="0 0 0" />
+            <origin xyz="0.3 0 -0.1" rpy="0 0 0" />
             <geometry>
                 <sphere radius="0.1" />
@@ -28,5 +28,5 @@
         </collision>
         <visual>
-            <origin xyz=" 0.3 0 0.1" rpy="0 0 0" />
+            <origin xyz=" 0.3 0 -0.1" rpy="0 0 0" />
             <geometry>
                 <sphere radius="0.1" />
@@ -34,5 +34,5 @@
         </visual>
         <visual>
-            <origin xyz="0.3 0 0.43" rpy="0 0 0" />
+            <origin xyz="0.3 0 0.23" rpy="0 0 0" />
             <geometry>
                 <cylinder radius="0.03" length="0.5" />
@@ -40,4 +40,9 @@
         </visual>
     </link>
+    <joint name="base_chassis_joint" type="fixed">
+        <parent link="base_link" />
+        <child link="chassis" />
+        <origin xyz="0 0 0.2" rpy="0 0 0" />
+    </joint>
     <link name="right_wheel">
         <inertial>
@@ -78,13 +83,9 @@
         </visual>
     </link>
-    <joint name="base_chassis_joint" type="fixed">
-        <parent link="base_link" />
-        <child link="chassis" />
-    </joint>
     <joint name="right_wheel_hinge" type="continuous">
         <parent link="chassis" />
         <child link="right_wheel" />
         <axis xyz="0 1 0" />
-        <origin xyz="-0.2 0.26 0.2" rpy="0 0 0" />
+        <origin xyz="-0.2 0.26 0" rpy="0 0 0" />
     </joint>
     <joint name="left_wheel_hinge" type="continuous">
@@ -92,5 +93,5 @@
         <child link="left_wheel" />
         <axis xyz="0 1 0" />
-        <origin xyz="-0.2 -0.26 0.2" rpy="0 0 0" />
+        <origin xyz="-0.2 -0.26 0" rpy="0 0 0" />
     </joint>
     <link name="camera">
@@ -114,6 +115,6 @@
     <joint name="camera_joint" type="fixed">
         <axis xyz="0 0 1" />
-        <origin xyz="0.35 0 0.6" rpy="0 0.5 0" />
-        <parent link="chassis"/>
+        <origin xyz="0.35 0 0.4" rpy="0 0.5 0" />
+        <parent link="chassis" />
         <child link="camera" />
     </joint>

Commit message: meshes

File: viratbot_description/urdf/viratbot.gazebo.xacro (robot description, xacro)
@@ -1,4 +1,7 @@
 <?xml version="1.0" encoding="UTF-8"?>
 <robot name="viratbot">
+    <gazebo reference="caster">
+        <material>Gazebo/Black</material>
+    </gazebo>
     <!-- Camera Plugin -->
     <gazebo reference="camera">
@@ -44,5 +47,5 @@
           <rightJoint>right_wheel_hinge</rightJoint>
           <wheelSeparation>0.52</wheelSeparation>
-          <wheelDiameter>0.4</wheelDiameter>
+          <wheelDiameter>0.28</wheelDiameter>
           <wheelAcceleration>1.0</wheelAcceleration>
           <wheelTorque>20</wheelTorque>
@@ -52,5 +55,5 @@
           <robotBaseFrame>base_link</robotBaseFrame>
           <odometrySource>1</odometrySource>
-          <publishWheelTF>true</publishWheelTF>
+          <!-- <publishWheelTF>true</publishWheelTF> -->
           <publishOdom>true</publishOdom>
           <publishWheelJointState>true</publishWheelJointState>

File: viratbot_description/urdf/viratbot.urdf.xacro (robot description, xacro)
@@ -3,12 +3,17 @@
     <xacro:include filename="$(find viratbot_description)/urdf/viratbot.gazebo.xacro" />
     <link name="base_link"></link>
+    <!-- Chassis -->
+    <xacro:property name="c_m" value="10" />
+    <xacro:property name="c_l" value="0.8" />
+    <xacro:property name="c_b" value="0.4" />
+    <xacro:property name="c_h" value="0.2" />
     <link name="chassis">
         <inertial>
-            <mass value="3" />
-            <inertia ixx="0.05" ixy="0" ixz="0" iyy="0.17" iyz="0" izz="0.2" />
+            <mass value="10" />
+            <inertia ixx="${((1/12)*c_m*(c_b*c_b + c_h*c_h)) + c_m*c_h/2*c_h/2}" ixy="0" ixz="0" iyy="${((1/12)*c_m*(c_l*c_l + c_h*c_h)) + c_m*c_h/2*c_h/2}" iyz="0" izz="${(1/12)*c_m*(c_b*c_b + c_l*c_l)}" />
             <origin xyz="0 0 0" rpy="0 0 0" />
         </inertial>
         <collision>
-            <origin rpy="0 0 0" xyz="0 0 0.2" />
+            <origin rpy="0 0 0" xyz="0 0 0.1" />
             <geometry>
                 <box size="0.8 0.4 0.2" />
@@ -16,25 +21,7 @@
         </collision>
         <visual>
-            <origin rpy=" 0 0 0" xyz="0 0 0" />
+            <origin rpy="0 0 0" xyz="-0.2 0 0" />
             <geometry>
-                <box size="0.8 0.4 0.2" />
-            </geometry>
-        </visual>
-        <collision>
-            <origin xyz="0.3 0 -0.1" rpy="0 0 0" />
-            <geometry>
-                <sphere radius="0.1" />
-            </geometry>
-        </collision>
-        <visual>
-            <origin xyz=" 0.3 0 -0.1" rpy="0 0 0" />
-            <geometry>
-                <sphere radius="0.1" />
-            </geometry>
-        </visual>
-        <visual>
-            <origin xyz="0.3 0 0.23" rpy="0 0 0" />
-            <geometry>
-                <cylinder radius="0.03" length="0.5" />
+                <mesh filename="package://viratbot_description/meshes/bot2.dae" scale="0.8 0.8 0.8" />
             </geometry>
         </visual>
@@ -43,10 +30,47 @@
         <parent link="base_link" />
         <child link="chassis" />
-        <origin xyz="0 0 0.2" rpy="0 0 0" />
+        <origin xyz="0 0 0.14" rpy="0 0 0" />
     </joint>
+    <!-- Caster Front -->
+    <xacro:property name="cas_m" value="0.3" />
+    <xacro:property name="cas_r" value="0.07" />
+    <link name="caster">
+        <inertial>
+            <mass value="${cas_m}" />
+            <inertia ixx="${(2/5)*cas_m*cas_r*cas_r}" ixy="0" ixz="0" iyy="${(2/5)*cas_m*cas_r*cas_r}" iyz="0" izz="${(2/5)*cas_m*cas_r*cas_r}" />
+        </inertial>
+        <collision>
+            <origin xyz="0 0 0" rpy="0 0 0" />
+            <geometry>
+                <sphere radius="0.07" />
+            </geometry>
+        </collision>
+        <visual>
+            <origin xyz="0 0 0" rpy="0 0 0" />
+            <geometry>
+                <sphere radius="0.07" />
+            </geometry>
+        </visual>
+        <visual>
+            <origin xyz="0 0 0.08" rpy="0 0 0" />
+            <geometry>
+                <cylinder radius="0.01" length="0.05" />
+            </geometry>
+        </visual>
+    </link>
+    <joint name="caster_chassis_joint" type="fixed">
+        <parent link="chassis" />
+        <child link="caster" />
+        <axis xyz="0 1 0" />
+        <origin xyz="0.2 0 -0.07" rpy="0 0 0" />
+    </joint>
+    <!-- Left ad Right Wheels -->
+    <xacro:property name="w_m" value="1" />
+    <xacro:property name="w_r" value="0.14" />
+    <xacro:property name="w_l" value="0.1" />
     <link name="right_wheel">
         <inertial>
-            <mass value="0.3" />
-            <inertia ixx="0.0325" ixy="0" ixz="0" iyy="0.006" iyz="0" izz="0.0325" />
+            <mass value="1" />
+            <inertia ixx="${(1/12)*w_m*(3*w_r*w_r + w_l*w_l)}" ixy="0" ixz="0" iyy="${(1/2)*w_m*w_r*w_r}" iyz="0" izz="${(1/12)*w_m*(3*w_r*w_r + w_l*w_l)}" />
             <origin xyz="0 0 0" rpy="0 1.5707 1.5707" />
         </inertial>
@@ -54,11 +78,11 @@
             <origin xyz="0 0 0" rpy="0 1.5707 1.5707" />
             <geometry>
-                <cylinder radius="0.2" length="0.1" />
+                <cylinder radius="0.14" length="0.1" />
             </geometry>
         </collision>
         <visual>
-            <origin xyz="0 0 0" rpy="0 1.5707 1.5705" />
+            <origin xyz="0 0 0" rpy="0 1.5707 0" />
             <geometry>
-                <cylinder radius="0.2" length="0.1" />
+                <mesh filename="package://viratbot_description/meshes/tyre1.dae" scale="1 1 1" />
             </geometry>
         </visual>
@@ -66,6 +90,6 @@
     <link name="left_wheel">
         <inertial>
-            <mass value="0.3" />
-            <inertia ixx="0.0325" ixy="0" ixz="0" iyy="0.006" iyz="0" izz="0.0325" />
+            <mass value="1" />
+            <inertia ixx="${(1/12)*w_m*(3*w_r*w_r + w_l*w_l)}" ixy="0" ixz="0" iyy="${(1/2)*w_m*w_r*w_r}" iyz="0" izz="${(1/12)*w_m*(3*w_r*w_r + w_l*w_l)}" />
             <origin xyz="0 0 0" rpy="0 1.5707 1.5707" />
         </inertial>
@@ -73,11 +97,11 @@
             <origin xyz="0 0 0" rpy="0 1.5707 1.5707" />
             <geometry>
-                <cylinder radius="0.2" length="0.1" />
+                <cylinder radius="0.14" length="0.1" />
             </geometry>
         </collision>
         <visual>
-            <origin xyz="0 0 0" rpy="0 1.5707 1.5705" />
+            <origin xyz="0 0 0" rpy="0 1.5707 0" />
             <geometry>
-                <cylinder radius="0.2" length="0.1" />
+                <mesh filename="package://viratbot_description/meshes/tyre1.dae" scale="1 1 1" />
             </geometry>
         </visual>
@@ -95,4 +119,5 @@
         <origin xyz="-0.2 -0.26 0" rpy="0 0 0" />
     </joint>
+    <!-- Camera -->
     <link name="camera">
         <inertial>
@@ -115,5 +140,5 @@
     <joint name="camera_joint" type="fixed">
         <axis xyz="0 0 1" />
-        <origin xyz="0.35 0 0.4" rpy="0 0.5 0" />
+        <origin xyz="0.43 0 0.4" rpy="0 0.5 0" />
         <parent link="chassis" />
         <child link="camera" />
