Commit message: camera

File: viratbot_description/urdf/viratbot.urdf.xacro (robot description, xacro)
@@ -24,4 +24,10 @@
             <geometry>
                 <sphere radius="0.1" />
+            </geometry>
+        </visual>
+        <visual>
+            <origin xyz="0.3 0 0.4" rpy="0 0 0"/>
+            <geometry>
+                <cylinder radius="0.03" length="0.8"/>
             </geometry>
         </visual>

Commit message: Added inertial elements

File: viratbot_description/urdf/viratbot.urdf.xacro (robot description, xacro)
@@ -1,5 +1,10 @@
-<?xml version="1.0" encoding="UTF-8"?>
+<?xml version="1.0"?>
 <robot name="viratbot" xmlns:xacro="http://www.ros.org/wiki/xacro">
-    <link name="chassis">
+    <link name="base_link">
+        <inertial>
+            <mass value="3"/>
+            <inertia ixx="0.05" ixy="0" ixz="0" iyy="0.17" iyz="0" izz="0.2"/>
+            <origin xyz="0 0 0.2" rpy="0 0 0"/>
+        </inertial>
         <collision>
             <origin rpy="0 0 0" xyz="0 0 0.2" />
@@ -15,5 +20,5 @@
         </visual>
         <collision>
-            <origin xyz=" -0.3 0 0.1" rpy="0 0 0" />
+            <origin xyz="0.3 0 0.1" rpy="0 0 0" />
             <geometry>
                 <sphere radius="0.1" />
@@ -27,13 +32,18 @@
         </visual>
         <visual>
-            <origin xyz="0.3 0 0.4" rpy="0 0 0"/>
+            <origin xyz="0.3 0 0.5" rpy="0 0 0" />
             <geometry>
-                <cylinder radius="0.03" length="0.8"/>
+                <cylinder radius="0.03" length="0.6" />
             </geometry>
         </visual>
     </link>
     <link name="right_wheel">
+        <inertial>
+            <mass value="0.3"/>
+            <inertia ixx="0.0325" ixy="0" ixz="0" iyy="0.006" iyz="0" izz="0.0325"/>
+            <origin xyz="0 0 0" rpy="0 1.5707 1.5707"/>
+        </inertial>
         <collision>
-            <origin xyz="-0.2 0.26 0.2" rpy="0 1.5707 1.5707"/>
+            <origin xyz="0 0 0" rpy="0 1.5707 1.5707" />
             <geometry>
                 <cylinder radius="0.2" length="0.1" />
@@ -41,5 +51,5 @@
         </collision>
         <visual>
-            <origin xyz="-0.2 0.26 0.2" rpy="0 1.5707 1.5705"/>
+            <origin xyz="0 0 0" rpy="0 1.5707 1.5705" />
             <geometry>
                 <cylinder radius="0.2" length="0.1" />
@@ -48,6 +58,11 @@
     </link>
     <link name="left_wheel">
+        <inertial>
+            <mass value="0.3"/>
+            <inertia ixx="0.0325" ixy="0" ixz="0" iyy="0.006" iyz="0" izz="0.0325"/>
+            <origin xyz="0 0 0" rpy="0 1.5707 1.5707"/>
+        </inertial>
         <collision>
-            <origin xyz="-0.2 -0.26 0.2" rpy="0 1.5707 1.5707"/>
+            <origin xyz="0 0 0" rpy="0 1.5707 1.5707" />
             <geometry>
                 <cylinder radius="0.2" length="0.1" />
@@ -55,5 +70,5 @@
         </collision>
         <visual>
-            <origin xyz="-0.2 -0.26 0.2" rpy="0 1.5707 1.5705"/>
+            <origin xyz="0 0 0" rpy="0 1.5707 1.5705" />
             <geometry>
                 <cylinder radius="0.2" length="0.1" />
@@ -62,10 +77,14 @@
     </link>
     <joint name="right_wheel_hinge" type="continuous">
-        <parent link="chassis" />
+        <parent link="base_link" />
         <child link="right_wheel" />
+        <axis xyz="0 1 0" />
+        <origin xyz="-0.2 0.26 0.2" rpy="0 0 0" />
     </joint>
     <joint name="left_wheel_hinge" type="continuous">
-        <parent link="chassis" />
+        <parent link="base_link" />
         <child link="left_wheel" />
+        <axis xyz="0 1 0" />
+        <origin xyz="-0.2 -0.26 0.2" rpy="0 0 0" />
     </joint>
 </robot>

Commit message: Publish Pothole coords

File: viratbot_description/urdf/viratbot.urdf.xacro (robot description, xacro)
@@ -140,7 +140,14 @@
     <joint name="camera_joint" type="fixed">
         <axis xyz="0 0 1" />
-        <origin xyz="0.43 0 0.4" rpy="0 0.5 0" />
+        <origin xyz="0.43 0 0.4" rpy="0 0.63 0" />
         <parent link="chassis" />
         <child link="camera" />
     </joint>
+    <!-- Frame for reference -->
+    <link name="camera_base"></link>
+    <joint name="camera_b_chassis" type="fixed">
+        <origin xyz="0.43 0 0" rpy="0 0 0" />
+        <parent link="base_link" />
+        <child link="camera_base" />
+    </joint>
 </robot>
